Commit message: added plots for fancy-looking pendulum

File: pendulum/pendulum.urdf (robot description, URDF)
Before this commit: robot pendulum, 2 links, 1 joints
Links:
- added link base, mass 0; visual sphere radius=0.1
- added link link_eef, mass 1; visual sphere radius=0.05
- link link_1: mass None -> 0; geometry visual cylinder length=0.8 radius=0.01
Joints:
- added joint joint_eef: type fixed, parent link_1, child link_eef, origin xyz=0 0 0.8 rpy=0 0 0
- added joint world_to_base: type fixed, parent world, child base, origin xyz=0 0 1 rpy=0 3.1415 0
- joint joint_1: origin xyz=0.0 0 0 rpy=0 0 0 -> xyz=0 0 0 rpy=0 0 0; parent world -> base

Commit message: lqr and feedback lin

File: pendulum/pendulum.urdf (robot description, URDF)
Before this commit: robot pendulum, 4 links, 3 joints
Joints:
- joint world_to_base: origin xyz=0 0 1 rpy=0 3.1415 0 -> xyz=0 0 1 rpy=0 3.141592653589793 0
